File: usb2seraialft8u232am.kicad_pcb (KiCad board)
At the start: 2 copper layers, 20 parts, among them P1 USB_A, P2 CONN_01X06, U1 FT232RQ, U2 MAX232

Commit message: new PCB design
Parts:
- C1, C11, C5, C6, C7, U2: moved to B.Cu
- P1: footprint Connect:USB_A -> auv:USB-A-PLUG_UDRA04MTKNN
- moved C1 37.4 mm to (136.7, 102.4), turned to 0 degrees
- moved P2 35.4 mm to (144.0, 101.6)
- moved C7 32.3 mm to (136.1, 112.8)
- moved U2 30.5 mm to (133.0, 107.1), turned to 90 degrees
- moved C11 29.2 mm to (129.8, 111.8), turned to 0 degrees
- moved C6 28.7 mm to (132.8, 111.8)
- moved C5 27.2 mm to (137.7, 112.8), turned to 270 degrees
- moved C10 25.8 mm to (126.0, 105.4), turned to 180 degrees
- moved C8 25.0 mm to (126.0, 109.7)
- moved C9 24.4 mm to (126.0, 107.7), turned to 180 degrees
- moved P1 21.9 mm to (120.7, 108.0)
- moved U1 21.2 mm to (131.8, 106.9), turned to 270 degrees
- moved C3 20.1 mm to (134.6, 102.9), turned to 180 degrees
- moved FB1 20.1 mm to (125.2, 112.5)
- moved R2 18.3 mm to (138.9, 110.7)
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Routing:
- net +5V: track 121.0 -> 53.4 mm, vias 7 -> 4
- net GND: track 60.4 -> 88.8 mm
- net Net-(P2-Pad6): track 39.5 -> 19.6 mm, vias 2 -> 0
- net Net-(C10-Pad1): track 27.4 -> 9.46 mm
- net /RxD: track 16.0 -> 4.00 mm, vias 2 -> 1
- net Net-(P2-Pad2): track 22.9 -> 11.0 mm
- net Net-(C8-Pad1): track 20.9 -> 9.13 mm, vias 2 -> 0
- net Net-(P2-Pad5): track 19.5 -> 27.4 mm
- net Net-(C9-Pad1): track 16.2 -> 9.98 mm
- net Net-(C7-Pad2): track 8.18 -> 2.23 mm, vias 2 -> 0
- net Net-(C5-Pad2): track 4.27 -> 9.86 mm
- net /~RTS~: track 8.27 -> 13.4 mm, vias 0 -> 1
- net /LEDRX: track 10.1 -> 5.07 mm
- net Net-(P2-Pad1): track 26.5 -> 21.7 mm
- net /~CTS~: track 8.47 -> 3.81 mm, vias 0 -> 1
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