File: usb2seraialft8u232am.sch (KiCad schematic (older format))
At the start: 21 parts, among them P1 USB_A, P2 CONN_01X06, U1 FT232RQ, U2 MAX232

Commit message: new PCB design
Parts:
- removed R1: R, Resistors_SMD:R_0603, symbol R
- P1: footprint Connect:USB_A -> auv:USB-A-PLUG_UDRA04MTKNN
Connections:
- wire segments 91 -> 90
Changed lines of the file:
@@
 LIBS:ft232bm
 LIBS:auv
-LIBS:usb2seraialft8u232am-cache
 EELAYER 25 0
 EELAYER END
@@
 F 0 "P1" H 1100 3450 50  0000 C CNN
 F 1 "USB_A" H 850 3850 50  0000 C CNN
-F 2 "Connect:USB_A" V 850 3550 50  0001 C CNN
+F 2 "auv:USB-A-PLUG_UDRA04MTKNN" V 850 3550 50  0001 C CNN
 F 3 "" V 850 3550 50  0000 C CNN
 	1    900  3650
@@
 $EndComp
 $Comp
-L R R1
-U 1 1 58025FD3
-P 10000 4050
-F 0 "R1" V 10080 4050 50  0000 C CNN
-F 1 "R" V 10000 4050 50  0000 C CNN
-F 2 "Resistors_SMD:R_0603" V 9930 4050 50  0001 C CNN
-F 3 "" H 10000 4050 50  0000 C CNN
-	1    10000 4050
-	0    1    1    0
-$EndComp
-$Comp
 L +5V #PWR015
 U 1 1 58026173
@@
 	9650 4550 9650 4050
 Wire Wire Line
-	9650 4050 9850 4050
-Wire Wire Line
-	10150 4050 10400 4050
+	9650 4050 10400 4050
 Wire Wire Line
 	10400 4050 10400 4000
